Commit message: fix axis orientation from bore detection phase

File: robots/UR5/robot.urdf (robot description, URDF)
Before this commit: robot UR5, 7 links, 6 joints
Joints:
- joint joint_2: axis 0 0 1 -> 0 1 0
- joint joint_3: axis 0 0 1 -> 0 1 0
- joint joint_4: axis 0 0 1 -> 0 1 0
- joint joint_5: axis 0 0 -1 -> 0 1 0
