Commit message: fix wrist2 joint axes and auto-propagate bore axes to chain.yaml
Joint 5/6 axes were swapped vs the UR5 spec (Z-Y-Y-Y-Z-Y). Fixed
chain.yaml, removed hardcoded joint_5 origin so it auto-computes from
the wrist1 distal bore, and added bore axis propagation in Save &
Rebuild so future Edit Bores changes update chain.yaml automatically.

Co-Authored-By: Claude Opus 4.6 <noreply@anthropic.com>

File: robots/UR5/robot.urdf (robot description, URDF)
Before this commit: robot UR5, 7 links, 6 joints
Joints:
- joint joint_5: axis 0 1 0 -> 0 0 1; origin xyz=0 0.093150 0 rpy=0 0 0 -> xyz=0.000205 0.095447 0.047500 rpy=0 0 0
- joint joint_6: axis 0 0 1 -> 0 1 0

Commit message: fix joint_6 origin: use auto-computed bore offsets instead of hardcoded DH
Removed the hardcoded origin override for joint_6 in chain.yaml so
the URDF generator computes it from wrist2's proximal/distal bore
positions. joint_6 now places wrist3 at wrist2's distal bore face.

Co-Authored-By: Claude Opus 4.6 <noreply@anthropic.com>

File: robots/UR5/robot.urdf (robot description, URDF)
Before this commit: robot UR5, 7 links, 6 joints
Joints:
- joint joint_6: origin xyz=0 0 0.094650 rpy=0 0 0 -> xyz=-0.001769 0.047596 0.047532 rpy=0 0 0

Commit message: fix: restore Meca500 end effector origin and UR5 wrist manual bores
The previous commit accidentally dropped the EndEffector visual origin
and overwrote the manually placed wrist1/2/3 connection points with
auto-detected ones.

Co-Authored-By: Claude Opus 4.6 <noreply@anthropic.com>

File: robots/UR5/robot.urdf (robot description, URDF)
Before this commit: robot UR5, 7 links, 6 joints
Joints:
- joint joint_5: origin xyz=0.001095 -0.045608 -0.046972 rpy=0 0 0 -> xyz=0.000205 0.095447 0.047500 rpy=0 0 0
- joint joint_6: origin xyz=-0.000483 -0.048289 -0.044500 rpy=0 0 0 -> xyz=-0.001769 0.047596 0.047532 rpy=0 0 0

Commit message: fix: use Z-position heuristic for proximal/distal on multi-axis parts
The multi-axis connection point detector previously assigned proximal/
distal labels based on cylinder length, which was unreliable for parts
with similar-length cylinders (e.g. UR5 wrists). Now assigns by
Z-position of the detected bore centers: lower Z = proximal (toward
base), higher Z = distal (toward tip), leveraging the Z-up STL
convention.

Also adds a largest-flat-face fallback in detect_base_connection for
parts with no Z-up faces (e.g. UR5 wrist3 end-effector flange).

Regenerated all robots except Meca500-R3 with --override-manual.

Co-Authored-By: Claude Opus 4.6 <noreply@anthropic.com>

File: robots/UR5/robot.urdf (robot description, URDF)
Before this commit: robot UR5, 7 links, 6 joints
Joints:
- joint joint_5: origin xyz=0.000205 0.095447 0.047500 rpy=0 0 0 -> xyz=-0.001095 0.045608 0.046972 rpy=0 0 0
- joint joint_6: origin xyz=-0.001769 0.047596 0.047532 rpy=0 0 0 -> xyz=0.000483 0.048289 0.044500 rpy=0 0 0

Commit message: fix: recompute derived joint origins after parent visual shifts
Connection-point-derived joint origins were calculated as
(distal − proximal) / 1000, which assumes the parent's proximal sits at
the frame origin.  When close_surface_gaps_along_axis later shifted the
parent's visual origin, the distal moved in the parent frame but the
downstream joint origin was never updated — producing ~41 mm placement
error on UR5 wrist2.

Add update_derived_joint_origins pass after surface gap closing to
recompute these origins using the finalized parent visual positions.

Co-Authored-By: Claude Opus 4.6 <noreply@anthropic.com>

File: robots/UR5/robot.urdf (robot description, URDF)
Before this commit: robot UR5, 7 links, 6 joints
Joints:
- joint joint_5: origin xyz=-0.001095 0.045608 0.046972 rpy=0 0 0 -> xyz=-0.001095 0.086609 0.046972 rpy=0 0 0

Commit message: Refine new robots: visual alignment, UX fixes, and docs (#29)
* redo make robot on all non Meca

* redo make-robots on 3 new robots with overwrite manual adjustments.

* fix: use Z-position heuristic for proximal/distal on multi-axis parts

The multi-axis connection point detector previously assigned proximal/
distal labels based on cylinder length, which was unreliable for parts
with similar-length cylinders (e.g. UR5 wrists). Now assigns by
Z-position of the detected bore centers: lower Z = proximal (toward
base), higher Z = distal (toward tip), leveraging the Z-up STL
convention.

Also adds a largest-flat-face fallback in detect_base_connection for
parts with no Z-up faces (e.g. UR5 wrist3 end-effector flange).

Regenerated all robots except Meca500-R3 with --override-manual.

Co-Authored-By: Claude Opus 4.6 <noreply@anthropic.com>

* fix: recompute derived joint origins after parent visual shifts

Connection-point-derived joint origins were calculated as
(distal − proximal) / 1000, which assumes the parent's proximal sits at
the frame origin.  When close_surface_gaps_along_axis later shifted the
parent's visual origin, the distal moved in the parent frame but the
downstream joint origin was never updated — producing ~41 mm placement
error on UR5 wrist2.

Add update_derived_joint_origins pass after surface gap closing to
recompute these origins using the finalized parent visual positions.

Co-Authored-By: Claude Opus 4.6 <noreply@anthropic.com>

* fix: use position-based proximal/distal in largest_face_fallback

The largest_face_fallback path in detect_base_connection hardcoded
end="distal", which misclassified wrist3's mating face as distal when
it should be proximal.  Now checks whether the face is at the min or
max end of its axis to determine the label — min = proximal, max = distal.

Fixes UR5 wrist3 placement (was offset in +Y due to missing proximal).

Co-Authored-By: Claude Opus 4.6 <noreply@anthropic.com>

* feat: auto-detect frame flips and all-barrel parts in connection detection

- Add auto_detect_visual_flips: when a joint's origin_rpy flips the child
  frame, anchor the visual on the distal connection point instead of
  proximal so the mesh extends in the correct world direction.
- Add all-barrel fallback in connections.py: when all cylinder groups have
  radii larger than the shortest bbox dimension, fall back to endpoint
  detection along the longest axis instead of multi-axis detection.
- Cap cross-section slice offsets for elongated parts (>200mm) so slices
  stay near end faces where bore openings are.
- Fixes Kinova-Gen3 shoulder positioning and bicep connection points
  (r≈20mm bore faces instead of r≈200mm barrel body).

Co-Authored-By: Claude Opus 4.6 <noreply@anthropic.com>

* fix: Move Part drag works on initial Edit Connections load

Default dragEnabled to true so it doesn't depend on the delayed
FACE_MARKER_INIT_JS timer firing before the UI init call. The
mousedown handler already gates on __faceEditMode, so drag only
activates inside Edit Connections mode.

Co-Authored-By: Claude Opus 4.6 <noreply@anthropic.com>

* fix: transform Move Part drag delta from world space to link-local frame

The drag delta from JS is in world space, but visual_xyz is applied in
the link's local frame. For frame-flipped links (e.g. Kinova shoulder
with π around X), Y and Z were inverted on rebuild. Now rotates the
delta by R_world^T before saving to chain.yaml.

Co-Authored-By: Claude Opus 4.6 <noreply@anthropic.com>

* feat: improve Edit Connections UX — camera-relative nudge and auto-show frames

Arrow keys now move parts along screen-relative axes with correct signs,
Shift modifier gives 2mm steps, and coordinate frames auto-enable on edit.

Co-Authored-By: Claude Opus 4.6 (1M context) <noreply@anthropic.com>

* fix: align Kinova Gen3 visual origins and clear connection points

Manually refined visual_xyz offsets for all Kinova links to achieve
full mesh alignment. Cleared auto-detected connection points that
were producing incorrect placements. Centered end effector mesh on
its rotation axis. Updated Edit Connections docs for Shift-nudge.

Co-Authored-By: Claude Opus 4.6 <noreply@anthropic.com>

* fix: center UR5 end effector mesh on its rotation axis

Zero out cross-axis (X, Z) visual origin offsets for wrist3/link_6,
keeping only the Y offset for axial positioning.

Co-Authored-By: Claude Opus 4.6 <noreply@anthropic.com>

* feat: center all UR5 meshes on rotation axes and add center-on-axis skill

Zero out cross-axis visual origin offsets for all UR5 links (shoulder
through wrist2), centering each mesh on its joint rotation axis. FK
and joint origins are unchanged.

Add center-on-axis skill documenting the procedure: read joint axes,
calculate cross-axis nudges, apply to chain.yaml, regenerate, verify.

Co-Authored-By: Claude Opus 4.6 <noreply@anthropic.com>

* fix: align FANUC LRMate200iD visual origins and clear connection points

Manually refined visual_xyz offsets for all FANUC links, centering
meshes on their rotation axes. Cleared auto-detected connection
points that were producing incorrect placements. FK unchanged:
50 → 330 → 35 → 335 → 80 mm.

Co-Authored-By: Claude Opus 4.6 <noreply@anthropic.com>

* fix: stop Save & Rebuild from deleting visual_xyz for non-moved dirty links

The elif branch in _save_and_rebuild deleted existing visual_xyz
entries when a link was in connection_dirty_links but had no drag
offset (e.g. just selected). This caused meshes to snap back to
origin on rebuild. Also refine FANUC visual offsets for links 3-6.

Co-Authored-By: Claude Opus 4.6 <noreply@anthropic.com>

* refactor: consolidate three simulator skills into control-simulator

Merge zoom-rotate-camera, set-visible-parts, and edit-connections-ui
into a single control-simulator skill with separate sub-guide files.
Update all doc references.

Co-Authored-By: Claude Opus 4.6 <noreply@anthropic.com>

* fix: accumulate keyboard nudge deltas to prevent loss between polls

Arrow-key nudges fired every ~30ms but Python polled __lastPartMove
every 200ms, so rapid keypresses overwrote each other and most deltas
were lost. Now accumulate into the existing entry when the link matches.

Co-Authored-By: Claude Opus 4.6 <noreply@anthropic.com>

* feat: align ABB-IRB2400 visual origins and clear connection points

Meshes positioned via visual_xyz nudges after removing auto-detected
connection points. All joint origins unchanged.

Co-Authored-By: Claude Opus 4.6 <noreply@anthropic.com>

---------

Co-authored-by: Claude Opus 4.6 <noreply@anthropic.com>

File: robots/UR5/robot.urdf (robot description, URDF)
Before this commit: robot UR5, 7 links, 6 joints
Joints:
- joint joint_5: origin xyz=0.000205 0.095447 0.047500 rpy=0 0 0 -> xyz=-0.001095 0.086609 0.046972 rpy=0 0 0
- joint joint_6: origin xyz=-0.001769 0.047596 0.047532 rpy=0 0 0 -> xyz=0.000483 0.048289 0.044500 rpy=0 0 0
