Commit message: 2nd iteration on URDF, using a real image to sim compare

File: robots/Meca500-R3/robot.urdf (robot description, URDF)
Before this commit: robot Meca500-R3, 7 links, 6 joints
Joints:
- joint joint_3: origin xyz=0 0 0.135 rpy=0 -1.5708 0 -> xyz=0 0 0.135 rpy=0 0 0

Commit message: further visual refinement

File: robots/Meca500-R3/robot.urdf (robot description, URDF)
Before this commit: robot Meca500-R3, 7 links, 6 joints
Joints:
- joint joint_4: origin xyz=0.038000 0 0.120000 rpy=0 0 0 -> xyz=0.038000 0 0.120000 rpy=0 -1.570800 0
- joint joint_6: origin xyz=0 0 0.070000 rpy=0 0 0 -> xyz=0.070000 0 0 rpy=0 0 0

Commit message: testing simpler face to face connections

File: robots/Meca500-R3/robot.urdf (robot description, URDF)
Before this commit: robot Meca500-R3, 7 links, 6 joints
Joints:
- joint joint_2: origin xyz=0.000000 0.000000 0.042000 rpy=0 0 0 -> xyz=-0.000419 -0.049821 0.036191 rpy=0 0 0
- joint joint_5: origin xyz=0.055000 0.000000 0.000000 rpy=0 0 0 -> xyz=0.058382 0.033858 -0.001709 rpy=0 0 0

File: robots/UR5/robot.urdf (robot description, URDF)
Before this commit: robot UR5, 7 links, 6 joints
Joints:
- joint joint_1: origin xyz=0.000000 0.000000 0.089159 rpy=0 0 0 -> xyz=-0.001408 0.004207 0.024002 rpy=0 0 0
- joint joint_2: origin xyz=0.000000 0.135850 0.000000 rpy=0.000000 1.570796 0.000000 -> xyz=-0.000820 0.064150 0.064174 rpy=0.000000 1.570796 0.000000
- joint joint_3: origin xyz=0.000000 -0.119700 0.425000 rpy=0 0 0 -> xyz=-0.002902 0.000000 0.430568 rpy=0 0 0
- joint joint_4: origin xyz=0.000000 0.000000 0.392250 rpy=0.000000 1.570796 0.000000 -> xyz=-0.000590 -0.006999 0.395787 rpy=0.000000 1.570796 0.000000
