Commit message: Add programmatic connection point detection and URDF generation pipeline
Replace manual URDF offset guessing with a two-stage pipeline:
analyze detects bore/shaft centers at mesh ends via cross-section
slicing, then generate computes exact transforms from a chain.yaml
kinematic spec. All 6 Meca500 joints validate at 0mm error.

New: ConnectionPoint model, connections.py, urdf_generator.py,
chain.yaml, generate CLI command, verify_kinematics --json mode.
Updated: assembly-reasoning skill, README with full project docs.

Co-Authored-By: Claude Opus 4.6 <noreply@anthropic.com>

File: robots/Meca500-R3/robot.urdf (robot description, URDF)
Before this commit: robot Meca500-R3, 7 links, 6 joints
Joints:
- joint joint_1: limit lower=-3.0543 upper=3.0543 effort=100 velocity=2.618 -> lower=-3.054 upper=3.054 effort=100 velocity=1; origin xyz=0 0 0.093 rpy=0 0 0 -> xyz=0 0 0.093000 rpy=0 0 0
- joint joint_2: limit lower=-1.2217 upper=1.5708 effort=100 velocity=2.618 -> lower=-1.2217 upper=1.5708 effort=100 velocity=1; origin xyz=0 0 0.042 rpy=0 0 0 -> xyz=0 0 0.042000 rpy=0 0 0
- joint joint_3: limit lower=-2.3562 upper=1.2217 effort=100 velocity=3.1416 -> lower=-2.3562 upper=1.2217 effort=100 velocity=1; origin xyz=0 0 0.135 rpy=0 0 0 -> xyz=0 0 0.135000 rpy=0 0 0
- joint joint_4: limit lower=-2.9671 upper=2.9671 effort=100 velocity=5.2360 -> lower=-2.9671 upper=2.9671 effort=100 velocity=1; origin xyz=0.038 0 0.120 rpy=0 0 0 -> xyz=0.038000 0 0.120000 rpy=0 0 0
- joint joint_5: limit lower=-2.0071 upper=2.0071 effort=100 velocity=5.2360 -> lower=-2.0071 upper=2.0071 effort=100 velocity=1
- joint joint_6: limit lower=-3.1416 upper=3.1416 effort=100 velocity=8.7266 -> lower=-3.1416 upper=3.1416 effort=100 velocity=1; origin xyz=0 0 0.070 rpy=0 0 0 -> xyz=0 0 0.070000 rpy=0 0 0

Commit message: Fix wrist connection: A5 attaches to front bore of A3_4
- Remove incorrect visual_xyz shifts on link_2 and link_3 that displaced
  meshes 39-40mm downward from their joint origins
- Move joint_4 origin to match A3_4 distal bore position [62, 0, 76]mm
- Remove origin_rpy frame rotation; use axis [1,0,0] directly for J4/J6
  so wrist extends horizontally along X from the front bore
- A5/A6 now correctly attach to the circular bore on A3_4's front face

Co-Authored-By: Claude Opus 4.6 <noreply@anthropic.com>

File: robots/Meca500-R3/robot.urdf (robot description, URDF)
Before this commit: robot Meca500-R3, 7 links, 6 joints
Joints:
- joint joint_4: axis 0 0 1 -> 1 0 0; origin xyz=0.038000 0 0.120000 rpy=0 -1.570800 0 -> xyz=0.062000 0 0.076000 rpy=0 0 0
- joint joint_6: axis 0 0 1 -> 1 0 0

Commit message: Fix J5 pivot: move A5 to link_4, J5 now pitches only A6
- Move A5 mesh from link_5 to link_4 so J4 forearm roll rotates A5+A6
- Make link_5 virtual — J5 pitch sits between A5 and A6
- Place J5 origin at A5 distal bore [81mm along X] (end of yoke)
- Co-locate J6 with J5 [origin 0,0,0] bringing A6 much closer to A5

Co-Authored-By: Claude Opus 4.6 <noreply@anthropic.com>

File: robots/Meca500-R3/robot.urdf (robot description, URDF)
Before this commit: robot Meca500-R3, 7 links, 6 joints
Links:
- link link_4: geometry visual mesh filename=stl_files/A5.stl scale=0.001 0.001 0.001
- link link_5: geometry 
Joints:
- joint joint_5: origin xyz=0 0 0 rpy=0 0 0 -> xyz=0.081000 0 0 rpy=0 0 0
- joint joint_6: origin xyz=0.070000 0 0 rpy=0 0 0 -> xyz=0 0 0 rpy=0 0 0

Commit message: Fix A6 position: place J5 at A5 pitch bearing, A6 bore as COR
- Move J5 origin to [48mm, 0, 0] at A5's Z-axis cylinder center
  (pitch bearing inside yoke jaws)
- Co-locate J6 with J5 at [0, 0, 0]
- Remove visual_xyz on A6 — auto-offset places proximal bore at
  joint origin, which is the correct center of rotation

Co-Authored-By: Claude Opus 4.6 <noreply@anthropic.com>

File: robots/Meca500-R3/robot.urdf (robot description, URDF)
Before this commit: robot Meca500-R3, 7 links, 6 joints
Joints:
- joint joint_5: origin xyz=0.081000 0 0 rpy=0 0 0 -> xyz=0.048000 0 0 rpy=0 0 0

Commit message: further visual refinement
- Lower A2 by 12mm so shoulder bore centers on J2 COR
- Shift A6 back 20mm so bore circle centers on COR inside A5 yoke
- Move J5 origin deeper into A5 yoke (48mm → 55mm) to hide A6 bore between jaws

Co-Authored-By: Claude Opus 4.6 <noreply@anthropic.com>

File: robots/Meca500-R3/robot.urdf (robot description, URDF)
Before this commit: robot Meca500-R3, 7 links, 6 joints
Joints:
- joint joint_5: origin xyz=0.048000 0 0 rpy=0 0 0 -> xyz=0.055000 0 0 rpy=0 0 0

Commit message: Fix A2, A3_4, and A5 vertical positioning to match manufacturer reference
A2 and A3_4 meshes were too high because visual_xyz adjustments were far
too conservative relative to their proximal bore depths (~32mm and ~40mm).
A5 and A6 were then floating above A3_4 because only visual_xyz was used
(which doesn't move the COR). Fixed by:

- A2 visual_xyz Z: -0.015 → -0.030 (flush with shoulder)
- A3_4 visual_xyz Z: -0.003 → -0.038 (flush with elbow)
- joint_4 origin Z: 0.076 → 0.038 (moves COR + A5/A6 down with chain)
- Removed A5 visual_xyz (COR shift handles positioning)
- Updated verify_kinematics.py expected positions for joint_4/5/6

Co-Authored-By: Claude Opus 4.6 <noreply@anthropic.com>

File: robots/Meca500-R3/robot.urdf (robot description, URDF)
Before this commit: robot Meca500-R3, 7 links, 6 joints
Joints:
- joint joint_4: origin xyz=0.062000 0 0.076000 rpy=0 0 0 -> xyz=0.062000 0 0.038000 rpy=0 0 0

Commit message: feat: add EndEffector to Meca500-R3 and fix visibility panel
- Add EndEffector.stl to URDF kinematic chain on link_6, aligned to
  A6's distal bore with rotation derived from actual surface normals
- Move A6 mesh from link_6 to link_5 so joint_6 rotates only the
  end-effector (tool roll), not the wrist housing
- Skip meshless links in Visible Parts panel (removes phantom link_5)
- Update chain.yaml to reflect new mesh assignments
- Add Chrome connector workflow documentation as an explanation page

Co-Authored-By: Claude Opus 4.6 <noreply@anthropic.com>

File: robots/Meca500-R3/robot.urdf (robot description, URDF)
Before this commit: robot Meca500-R3, 7 links, 6 joints
Links:
- link link_5: geometry visual mesh filename=stl_files/A6.stl scale=0.001 0.001 0.001
- link link_6: geometry visual mesh filename=stl_files/EndEffector.stl scale=0.001 0.001 0.001

Commit message: feat: add three centering modes for bore visual origin alignment
Introduces surface_bbox (default), surface, and center centering modes
to handle different part geometries when aligning bore markers to DH
pivot points. Replaces the boolean center flag with a centering dropdown
in the Edit Bores UI. Closes visual gaps on UR5 while preserving Meca500
alignment.

Co-Authored-By: Claude Opus 4.6 <noreply@anthropic.com>

File: robots/Meca500-R3/robot.urdf (robot description, URDF)
Before this commit: robot Meca500-R3, 7 links, 6 joints
Joints:
- joint joint_1: axis 0 0 1 -> 0.000000 0.000000 1.000000; origin xyz=0 0 0.093000 rpy=0 0 0 -> xyz=0.000000 0.000000 0.093000 rpy=0 0 0
- joint joint_2: axis 0 1 0 -> 0.000000 1.000000 0.000000; origin xyz=0 0 0.042000 rpy=0 0 0 -> xyz=0.000000 0.000000 0.042000 rpy=0 0 0
- joint joint_3: axis 0 1 0 -> 0.000000 1.000000 0.000000; origin xyz=0 0 0.135000 rpy=0 0 0 -> xyz=0.000000 0.000000 0.135000 rpy=0 0 0
- joint joint_4: axis 1 0 0 -> 1.000000 0.000000 0.000000; origin xyz=0.062000 0 0.038000 rpy=0 0 0 -> xyz=0.062000 0.000000 0.038000 rpy=0 0 0
- joint joint_5: axis 0 1 0 -> 0.000000 1.000000 0.000000; origin xyz=0.055000 0 0 rpy=0 0 0 -> xyz=0.055000 0.000000 0.000000 rpy=0 0 0
- joint joint_6: axis 1 0 0 -> 1.000000 0.000000 0.000000; origin xyz=0 0 0 rpy=0 0 0 -> xyz=0.000000 0.000000 0.000000 rpy=0 0 0

File: robots/UR5/robot.urdf (robot description, URDF)
Before this commit: robot UR5, 7 links, 6 joints
Joints:
- joint joint_1: axis 0 0 1 -> 0.000000 0.000000 1.000000; origin xyz=0 0 0.089159 rpy=0 0 0 -> xyz=0.000000 0.000000 0.089159 rpy=0 0 0
- joint joint_2: axis 0 1 0 -> 0.000000 1.000000 0.000000; origin xyz=0 0.135850 0 rpy=0 1.570796 0 -> xyz=0.000000 0.135850 0.000000 rpy=0.000000 1.570796 0.000000
- joint joint_3: axis 0 1 0 -> 0.000000 1.000000 0.000000; origin xyz=0 -0.119700 0.425000 rpy=0 0 0 -> xyz=0.000000 -0.119700 0.425000 rpy=0 0 0
- joint joint_4: axis 0 1 0 -> 0.000000 1.000000 0.000000; origin xyz=0 0 0.392250 rpy=0 1.570796 0 -> xyz=0.000000 0.000000 0.392250 rpy=0.000000 1.570796 0.000000
- joint joint_5: axis 0 0 1 -> 0.000000 0.000000 1.000000; origin xyz=0.000205 0.095447 0.047500 rpy=0 0 0 -> xyz=0.001095 -0.045608 -0.046972 rpy=0 0 0
- joint joint_6: axis 0 1 0 -> 0.000000 1.000000 0.000000; origin xyz=-0.001769 0.047596 0.047532 rpy=0 0 0 -> xyz=-0.000483 -0.048289 -0.044500 rpy=0 0 0

Commit message: refactor: simplify surface centering — raw position, no adjustment
Surface mode now uses the raw proximal position with no centering
heuristic, and compute_joint_origin is left unchanged (DH-first).
Meca500 looks correct; UR5 surface gaps remain to be closed via
visual origin improvements.

Also persists EndEffector visual_xyz/rpy in Meca500 chain.yaml
and adds CLAUDE.md rule: never modify compute_joint_origin for
visual alignment.

Co-Authored-By: Claude Opus 4.6 <noreply@anthropic.com>

File: robots/Meca500-R3/robot.urdf (robot description, URDF)
Before this commit: robot Meca500-R3, 7 links, 6 joints
Joints:
- joint joint_2: origin xyz=-0.000419 -0.049821 0.036191 rpy=0 0 0 -> xyz=0.000000 0.000000 0.042000 rpy=0 0 0
- joint joint_5: origin xyz=0.058382 0.033858 -0.001709 rpy=0 0 0 -> xyz=0.055000 0.000000 0.000000 rpy=0 0 0

File: robots/UR5/robot.urdf (robot description, URDF)
Before this commit: robot UR5, 7 links, 6 joints
Joints:
- joint joint_1: origin xyz=-0.001408 0.004207 0.024002 rpy=0 0 0 -> xyz=0.000000 0.000000 0.089159 rpy=0 0 0
- joint joint_2: origin xyz=-0.000820 0.064150 0.064174 rpy=0.000000 1.570796 0.000000 -> xyz=0.000000 0.135850 0.000000 rpy=0.000000 1.570796 0.000000
- joint joint_3: origin xyz=-0.002902 0.000000 0.430568 rpy=0 0 0 -> xyz=0.000000 -0.119700 0.425000 rpy=0 0 0
- joint joint_4: origin xyz=-0.000590 -0.006999 0.395787 rpy=0.000000 1.570796 0.000000 -> xyz=0.000000 0.000000 0.392250 rpy=0.000000 1.570796 0.000000
